File: 16seg_Controller.kicad_pcb (KiCad board)
At the start: 2 copper layers, 64 x 72 mm, 59 parts, among them J1 Power, J2 USB, J3 Fan 1, J4 Fan 2, J5 Display, J6 LMJ2018814100DT1, Q1 BC807, Q2 BC807, U1 CH330N, U2 74HCT541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

Commit message: Fix missing paste on crystal pads
Parts:
- Y1: footprint Crystals:Crystal_SMD_TXC_7M-4pin_3.2x2.5mm -> custom:Crystal_4pin_3.2x2.5mm
Changed lines of the file:
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@@
     )
   )
-  (footprint "Crystals:Crystal_SMD_TXC_7M-4pin_3.2x2.5mm" (layer "F.Cu")
+  (footprint "custom:Crystal_4pin_3.2x2.5mm" (layer "F.Cu")
     (at 89 97.7 -90)
     (descr "SMD Crystal TXC 7M http://www.txccrystal.com/images/pdf/7m-accuracy.pdf, 3.2x2.5mm^2 package")
@@
     (property "Sheetname" "W5500 Ethernet")
     (attr smd)
-    (fp_text reference "Y1" (at 2.55 0.75 180) (layer "F.SilkS")
+    (fp_text reference "Y1" (at 2.55 0.75) (layer "F.SilkS")
       (effects (font (size 0.75 0.75) (thickness 0.1)))
     )
-    (fp_text value "25 MHz" (at 0 2.45 90) (layer "F.Fab")
+    (fp_text value "25 MHz" (at 0 2.45 -90) (layer "F.Fab")
       (effects (font (size 1 1) (thickness 0.15)))
     )
@@
     (fp_line (start -2 1.65) (end 2 1.65) (layer "F.SilkS") (width 0.12))
     (fp_line (start 2.1 1.7) (end 2.1 -1.7) (layer "F.CrtYd") (width 0.05))
+    (fp_line (start -2.1 1.7) (end 2.1 1.7) (layer "F.CrtYd") (width 0.05))
     (fp_line (start -2.1 -1.7) (end -2.1 1.7) (layer "F.CrtYd") (width 0.05))
     (fp_line (start 2.1 -1.7) (end -2.1 -1.7) (layer "F.CrtYd") (width 0.05))
-    (fp_line (start -2.1 1.7) (end 2.1 1.7) (layer "F.CrtYd") (width 0.05))
     (fp_line (start 1.6 1.25) (end 1.6 -1.25) (layer "F.Fab") (width 0.1))
+    (fp_line (start 1.6 -1.25) (end -1.6 -1.25) (layer "F.Fab") (width 0.1))
+    (fp_line (start -1.6 0.25) (end -0.6 1.25) (layer "F.Fab") (width 0.1))
+    (fp_line (start -1.6 -1.25) (end -1.6 1.25) (layer "F.Fab") (width 0.1))
     (fp_line (start -1.6 1.25) (end 1.6 1.25) (layer "F.Fab") (width 0.1))
-    (fp_line (start -1.6 -1.25) (end -1.6 1.25) (layer "F.Fab") (width 0.1))
-    (fp_line (start -1.6 0.25) (end -0.6 1.25) (layer "F.Fab") (width 0.1))
-    (fp_line (start 1.6 -1.25) (end -1.6 -1.25) (layer "F.Fab") (width 0.1))
-    (pad "1" smd rect locked (at -1.1 0.85 270) (size 1.4 1.2) (layers "F.Cu" "F.Mask")
+    (pad "1" smd rect locked (at -1.1 0.85 270) (size 1.4 1.2) (layers "F.Cu" "F.Paste" "F.Mask")
       (net 43 "Net-(C16-Pad2)") (pinfunction "1"))
-    (pad "2" smd rect locked (at 1.1 0.85 270) (size 1.4 1.2) (layers "F.Cu" "F.Mask")
+    (pad "2" smd rect locked (at 1.1 0.85 270) (size 1.4 1.2) (layers "F.Cu" "F.Paste" "F.Mask")
       (net 2 "GND") (pinfunction "2"))
-    (pad "3" smd rect locked (at 1.1 -0.85 270) (size 1.4 1.2) (layers "F.Cu" "F.Mask")
+    (pad "3" smd rect locked (at 1.1 -0.85 270) (size 1.4 1.2) (layers "F.Cu" "F.Paste" "F.Mask")
       (net 44 "Net-(C17-Pad1)") (pinfunction "3"))
-    (pad "4" smd rect locked (at -1.1 -0.85 270) (size 1.4 1.2) (layers "F.Cu" "F.Mask")
+    (pad "4" smd rect locked (at -1.1 -0.85 270) (size 1.4 1.2) (layers "F.Cu" "F.Paste" "F.Mask")
       (net 2 "GND") (pinfunction "4"))
-    (model "Crystals.3dshapes/Crystal_SMD_TXC_7M-4pin_3.2x2.5mm.wrl"
+    (model "${KIWALTER3DMOD}/Crystal IQXC-42.stp"
       (offset (xyz 0 0 0))
-      (scale (xyz 1 1 1))
+      (scale (xyz 1.6 1.6 1))
       (rotate (xyz 0 0 0))
     )
-    (model "${KIWALTER3DMOD}/Crystal IQXC-42.stp"
-      (offset (xyz 0 0 0))
-      (scale (xyz 1.7 1.7 1.7))
-      (rotate (xyz 0 0 0))
-    )
